File: SafeMiner.kicad_pcb (KiCad board)
At the start: 2 copper layers, 56.5 x 99.8 mm, 26 parts, among them J1 282837-2, Q1 FLAME SENSOR

Commit message: Add files via upload
Connections:
- C1 pad 2: VCC -> GND
- J1 pad 1: VCC -> GND (x5)
- J1 pad 2: GND -> VCC (x5)
- Q1 pad 1: VCC -> GND
- R1 pad 1: GND -> VCC
- RV1 pad 2: VCC -> GND
- RV1 pad 3: VCC -> GND
- gate pad 3: GND -> VCC
- gate pad Pin 2 power: VCC -> GND
Routing:
- net VCC: track 230.4 -> 147.0 mm
- net GND: track 146.5 -> 204.0 mm
Changed lines of the file:
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@@
 	(net 2 "Net-C1")
 	(net 3 "Net-D1")
-	(net 4 "VCC")
+	(net 4 "GND")
 	(net 5 "Net-Fire-Signal-Shutoff")
-	(net 6 "GND")
+	(net 6 "VCC")
 	(footprint "TerminalBlock:TerminalBlock_bornier-2_P5.08mm"
 		(layer "F.Cu")
@@
 			(layers "*.Cu" "*.Mask")
 			(remove_unused_layers no)
-			(net 4 "VCC")
+			(net 4 "GND")
 			(pinfunction "Pin_1")
 			(pintype "passive")
@@
 			(layers "*.Cu" "*.Mask")
 			(remove_unused_layers no)
-			(net 6 "GND")
+			(net 6 "VCC")
 			(pinfunction "Pin_2")
 			(pintype "passive")
@@
 			(layers "*.Cu" "*.Mask")
 			(remove_unused_layers no)
-			(net 4 "VCC")
+			(net 4 "GND")
 			(pinfunction "Pin_1")
 			(pintype "passive")
@@
 			(layers "*.Cu" "*.Mask")
 			(remove_unused_layers no)
-			(net 6 "GND")
+			(net 6 "VCC")
 			(pinfunction "Pin_2")
 			(pintype "passive")
@@
 			(layers "*.Cu" "*.Mask")
 			(remove_unused_layers no)
-			(net 6 "GND")
+			(net 6 "VCC")
 		)
 		(pad "2" thru_hole oval
@@
 			(layers "*.Cu" "*.Mask")
 			(remove_unused_layers no)
-			(net 4 "VCC")
+			(net 4 "GND")
 			(pinfunction "E")
 			(pintype "passive")
@@
 			(layers "*.Cu" "*.Mask")
 			(remove_unused_layers no)
-			(net 4 "VCC")
+			(net 4 "GND")
 			(pinfunction "Pin_1")
 			(pintype "passive")
@@
 			(layers "*.Cu" "*.Mask")
 			(remove_unused_layers no)
-			(net 6 "GND")
+			(net 6 "VCC")
 			(pinfunction "Pin_2")
 			(pintype "passive")
@@
 			(layers "*.Cu" "*.Mask")
 			(remove_unused_layers no)
-			(net 4 "VCC")
+			(net 4 "GND")
 			(pinfunction "Pin_1")
 			(pintype "passive")
@@
 			(layers "*.Cu" "*.Mask")
 			(remove_unused_layers no)
-			(net 6 "GND")
+			(net 6 "VCC")
 			(pinfunction "Pin_2")
 			(pintype "passive")
@@
 			(layers "*.Cu" "*.Mask")
 			(remove_unused_layers no)
-			(net 4 "VCC")
+			(net 4 "GND")
 			(pinfunction "2")
 			(pintype "passive")
@@
 			(layers "*.Cu" "*.Mask")
 			(remove_unused_layers no)
-			(net 4 "VCC")
+			(net 4 "GND")
 			(pinfunction "3")
 			(pintype "passive")
@@
 			(layers "*.Cu" "*.Mask")
 			(remove_unused_layers no)
-			(net 4 "VCC")
+			(net 4 "GND")
 			(pinfunction "Pin_1")
 			(pintype "passive")
@@
 			(layers "*.Cu" "*.Mask")
 			(remove_unused_layers no)
-			(net 6 "GND")
+			(net 6 "VCC")
 			(pinfunction "Pin_2")
 			(pintype "passive")
@@
 			(layers "*.Cu" "*.Mask")
 			(remove_unused_layers no)
-			(net 4 "VCC")
+			(net 4 "GND")
 			(pintype "passive")
 		)
@@
 			(layers "*.Cu" "*.Mask")
 			(remove_unused_layers no)
-			(net 6 "GND")
+			(net 6 "VCC")
 		)
 		(pad "Pin 1 Gate" thru_hole rect
@@
 			(layers "*.Cu" "*.Mask")
 			(remove_unused_layers no)
-			(net 4 "VCC")
+			(net 4 "GND")
 		)
 		(model "${KICAD8_3DMODEL_DIR}/Package_TO_SOT_THT.3dshapes/TO-220-3_Horizontal_TabDown.wrl"
@@
 	)
 	(segment
-		(start 126.4 88.6)
-		(end 115.6 99.4)
-		(width 2)
-		(layer "B.Cu")
-		(net 4)
-	)
-	(segment
 		(start 119.4 48.8)
 		(end 115.8 52.4)
@@
 	)
 	(segment
-		(start 115.6 99.4)
-		(end 104.4 99.4)
-		(width 2)
-		(layer "B.Cu")
-		(net 4)
-	)
-	(segment
 		(start 126.2 88.8)
 		(end 126 89)
@@
 	)
 	(segment
-		(start 129.66 48.8)
-		(end 128.26 48.8)
+		(start 112.92 94.2)
+		(end 99.4 94.2)
 		(width 2)
 		(layer "F.Cu")
@@
 	)
 	(segment
-		(start 124.06 83.2)
-		(end 105.52 83.2)
+		(start 123.92 83.2)
+		(end 112.92 94.2)
 		(width 2)
 		(layer "F.Cu")
@@
 	)
 	(segment
-		(start 98.8 95.6)
+		(start 98.8 94.8)
 		(end 98.8 104.28)
 		(width 2)
@@
 	)
 	(segment
-		(start 100.2 94.2)
-		(end 98.8 95.6)
+		(start 129.66 48.8)
+		(end 128.26 48.8)
+		(width 2)
+		(layer "F.Cu")
+		(net 6)
+	)
+	(segment
+		(start 124.06 83.2)
+		(end 105.52 83.2)
 		(width 2)
 		(layer "F.Cu")
@@
 	)
 	(segment
-		(start 123.92 83.2)
-		(end 112.92 94.2)
+		(start 99.4 94.2)
+		(end 98.8 94.8)
 		(width 2)
 		(layer "F.Cu")
@@
 		(width 2)
 		(layer "F.Cu")
-		(net 6)
-	)
-	(segment
-		(start 112.92 94.2)
-		(end 100.2 94.2)
-		(width 2)
-		(layer "F.Cu")
